File: Kicad/Gas_sensor_shield/Gas_sensor_shield.kicad_pcb (KiCad board)
At the start: 2 copper layers, 68.6 x 53.3 mm, 8 parts, among them P1 Power, P2 Analog, P3 Digital, P4 Digital, P5 CONN_01X01, P6 CONN_01X01, P7 CONN_01X01, P8 CONN_01X01

Commit message: Added the design of the electronic card
Parts:
- added C1: 100n, Capacitor_THT:CP_Radial_D5.0mm_P2.00mm, F.Cu at (166.8, 97.8)
- added C2: 1u, Capacitor_THT:CP_Radial_D5.0mm_P2.00mm, F.Cu at (166.9, 107.3)
- added C3: 100n, Capacitor_THT:CP_Radial_D5.0mm_P2.00mm, F.Cu at (166.9, 87.6)
- added C4: 100n, Capacitor_THT:CP_Radial_D5.0mm_P2.00mm, F.Cu at (158.5, 107.3)
- added D1: LED, LED_THT:LED_D3.0mm, F.Cu at (147.8, 91.4)
- added R1: 10k, Resistor_THT:R_Axial_DIN0204_L3.6mm_D1.6mm_P7.62mm_Horizontal, F.Cu at (128.8, 99.1)
- added R2: 100, Resistor_THT:R_Axial_DIN0204_L3.6mm_D1.6mm_P7.62mm_Horizontal, F.Cu at (128.8, 105.4)
- added R3: 100k, Resistor_THT:R_Axial_DIN0204_L3.6mm_D1.6mm_P7.62mm_Horizontal, F.Cu at (128.8, 111.8)
- added R4: 1k, Resistor_THT:R_Axial_DIN0204_L3.6mm_D1.6mm_P7.62mm_Horizontal, F.Cu at (128.8, 118.1)
- added R5: 100k, Resistor_THT:R_Axial_DIN0204_L3.6mm_D1.6mm_P7.62mm_Horizontal, F.Cu at (155.2, 114.6)
- added R6: 1k, Resistor_THT:R_Axial_DIN0204_L3.6mm_D1.6mm_P7.62mm_Horizontal, F.Cu at (165.7, 114.6)
- added R7: 1k, Resistor_THT:R_Axial_DIN0204_L3.6mm_D1.6mm_P7.62mm_Horizontal, F.Cu at (142.7, 99.1)
- added R8: 330, Resistor_THT:R_Axial_DIN0204_L3.6mm_D1.6mm_P7.62mm_Horizontal, F.Cu at (142.7, 105.4)
- added R9: 1k, Resistor_THT:R_Axial_DIN0204_L3.6mm_D1.6mm_P7.62mm_Horizontal, F.Cu at (150.4, 84.5)
- added U1: LTC1050, My_Package:LTC1050, F.Cu at (162.4, 92.7)
- added U2: Gas_Sensor, My_Package:Sensor_gas, F.Cu at (130.0, 88.3)
- added U3: RN2483_Breakout, My_Package:RN2483_breakout, F.Cu at (114.8, 108.6)
Connections:
- net /0(Rx) renamed /D0(Rx)
- net /1(Tx) renamed /D1(Tx)
- net /13(SCK) renamed /D13(SCK)
- net /2 renamed /D2
- net /3(**) renamed /D3(**)
- net /4 renamed /D4
- net /5(**) renamed /D5(**)
- net /6(**) renamed /D6(**)
- net /9(**) renamed /D9
- net /Reset renamed /~Reset~
- P3 pad 1: /A5(SCL) -> Net-(P3-Pad1)
- P3 pad 10: /8 -> /D8
- P3 pad 2: /A4(SDA) -> Net-(P3-Pad2)
- P3 pad 6: /12(MISO) -> /D12
- P3 pad 7: /11(**/MOSI) -> /D11
- P3 pad 8: /10(**/SS) -> /D10
- P4 pad 1: /7 -> /A1
Routing:
- added copper zone on F.Cu, net +5V
- added copper zone on B.Cu, net GND
