File: Kicad/Gas_sensor_shield/Gas_sensor_shield.sch (KiCad schematic (older format))
At the start: 22 parts, among them P1 Power, P2 Analog, P3 Digital, P4 Digital, P5 CONN_01X01, P6 CONN_01X01, P7 CONN_01X01, P8 CONN_01X01

Commit message: Added Design of the circuit board
Parts:
- removed U?: LTC1100xN8, Package_DIP:DIP-8_W7.62mm, symbol Amplifier_Instrumentation:LTC1100xN8
- added J1: Conn_01x02_Female, symbol Connector:Conn_01x02_Female
- added R2: R, symbol Device:R
- added U1: LTC1050, symbol My_Library:LTC1050
- added U2: Gas_Sensor, symbol My_Library:Gas_Sensor
- added U3: RN2483_Breakout, symbol My_Library:RN2483_Breakout
- R9: renamed from R?; value R -> 1k
- gave numbers to parts that had none: 12
Connections:
- net labels added: +3V3, D10, D11, D12, D9
- wire segments 82 -> 99
- no-connect marks 31 -> 34
Other:
- moved on the sheet: C1, C2, C3, C4, R1, R3, R4, R5, R6

Commit message: Added the design of the electronic card
Parts:
- removed J1: Conn_01x02_Female, symbol Connector:Conn_01x02_Female
- C1, C2, C3, C4: footprint (none) -> Capacitor_THT:CP_Radial_D5.0mm_P2.00mm
- D1: footprint (none) -> LED_THT:LED_D3.0mm
- R1, R3, R4, R5, R6, R7, R8, R9: footprint (none) -> Resistor_THT:R_Axial_DIN0204_L3.6mm_D1.6mm_P7.62mm_Horizontal
- R2: value R -> 100; footprint (none) -> Resistor_THT:R_Axial_DIN0204_L3.6mm_D1.6mm_P7.62mm_Horizontal
- U1: footprint (none) -> My_Package:LTC1050
- U2: footprint (none) -> My_Package:Sensor_gas
- U3: footprint (none) -> My_Package:RN2483_breakout
Connections:
- net D7 is gone; now on net A1: P4.1 (Pin_1)
- net +5V: now also U2.3 (Heater_1)

Commit message: modified the circuit board and routed
Parts:
- removed R7: 1k, Resistor_THT:R_Axial_DIN0204_L3.6mm_D1.6mm_P7.62mm_Horizontal, symbol Device:R
- removed R8: 330, Resistor_THT:R_Axial_DIN0204_L3.6mm_D1.6mm_P7.62mm_Horizontal, symbol Device:R
- added RV1: R_POT, Potentiometer_THT:Potentiometer_ACP_CA9-V10_Vertical, symbol Device:R_POT
- renumbered R9 to R7
Connections:
- net +5V: now also RV1.1
- net D6(**): now also RV1.2
- net GND: now also RV1.3
- no-connect marks 34 -> 33
Changed lines of the file:
@@
 $EndDescr
 $Comp
-L power:GND #PWR010
+L power:GND #PWR011
 U 1 1 5FCCB259
 P 7050 800
-F 0 "#PWR010" H 7050 550 50  0001 C CNN
+F 0 "#PWR011" H 7050 550 50  0001 C CNN
 F 1 "GND" H 7050 650 50  0000 C CNN
 F 2 "" H 7050 800 50  0000 C CNN
@@
 $EndComp
 $Comp
-L power:+3.3V #PWR013
+L power:+3.3V #PWR014
 U 1 1 5FCCD66D
 P 7600 800
-F 0 "#PWR013" H 7600 650 50  0001 C CNN
+F 0 "#PWR014" H 7600 650 50  0001 C CNN
 F 1 "+3.3V" V 7600 1050 50  0000 C CNN
 F 2 "" H 7600 800 50  0000 C CNN
@@
 $EndComp
 $Comp
-L power:+5V #PWR014
+L power:+5V #PWR015
 U 1 1 5FCCF251
 P 8150 800
-F 0 "#PWR014" H 8150 650 50  0001 C CNN
+F 0 "#PWR015" H 8150 650 50  0001 C CNN
 F 1 "+5V" V 8150 1000 50  0000 C CNN
 F 2 "" H 8150 800 50  0000 C CNN
@@
 $EndComp
 $Comp
-L power:GND #PWR019
+L power:GND #PWR020
 U 1 1 56D70CFF
 P 10300 3150
-F 0 "#PWR019" H 10300 2900 50  0001 C CNN
+F 0 "#PWR020" H 10300 2900 50  0001 C CNN
 F 1 "GND" H 10300 3000 50  0000 C CNN
 F 2 "" H 10300 3150 50  0000 C CNN
@@
 $EndComp
 $Comp
-L power:GND #PWR017
+L power:GND #PWR018
 U 1 1 56D70CC2
 P 9300 3150
-F 0 "#PWR017" H 9300 2900 50  0001 C CNN
+F 0 "#PWR018" H 9300 2900 50  0001 C CNN
 F 1 "GND" H 9300 3000 50  0000 C CNN
 F 2 "" H 9300 3150 50  0000 C CNN
@@
 $EndComp
 $Comp
-L power:+5V #PWR015
+L power:+5V #PWR016
 U 1 1 56D707BB
 P 9050 1350
-F 0 "#PWR015" H 9050 1200 50  0001 C CNN
+F 0 "#PWR016" H 9050 1200 50  0001 C CNN
 F 1 "+5V" V 9050 1550 50  0000 C CNN
 F 2 "" H 9050 1350 50  0000 C CNN
@@
 $EndComp
 $Comp
-L power:+3.3V #PWR016
+L power:+3.3V #PWR017
 U 1 1 56D70538
 P 9150 1450
-F 0 "#PWR016" H 9150 1300 50  0001 C CNN
+F 0 "#PWR017" H 9150 1300 50  0001 C CNN
 F 1 "+3.3V" V 9150 1700 50  0000 C CNN
 F 2 "" H 9150 1450 50  0000 C CNN
@@
 	4000 2150 4300 2150
 $Comp
-L power:+5V #PWR04
+L power:+5V #PWR05
 U 1 1 5FDF0C95
 P 4300 2150
-F 0 "#PWR04" H 4300 2000 50  0001 C CNN
+F 0 "#PWR05" H 4300 2000 50  0001 C CNN
 F 1 "+5V" H 4315 2323 50  0000 C CNN
 F 2 "" H 4300 2150 50  0001 C CNN
@@
 	9950 4850 9950 4600
 $Comp
-L power:GND #PWR018
+L power:GND #PWR019
 U 1 1 5FE609EC
 P 9950 6050
-F 0 "#PWR018" H 9950 5800 50  0001 C CNN
+F 0 "#PWR019" H 9950 5800 50  0001 C CNN
 F 1 "GND" H 9955 5877 50  0000 C CNN
 F 2 "" H 9950 6050 50  0001 C CNN
@@
 $EndComp
 $Comp
-L Device:R R9
+L Device:R R7
 U 1 1 5FE567CC
 P 9950 5000
-F 0 "R9" H 10020 5046 50  0000 L CNN
+F 0 "R7" H 10020 5046 50  0000 L CNN
 F 1 "1k" H 10020 4955 50  0000 L CNN
 F 2 "Resistor_THT:R_Axial_DIN0204_L3.6mm_D1.6mm_P7.62mm_Horizontal" V 9880 5000 50  0001 C CNN
@@
 	1    0    0    -1
 $EndComp
-Text Label 7850 5350 0    50   ~ 0
-D6
-Wire Wire Line
-	7350 5350 7350 5150
-Connection ~ 7350 5350
-Wire Wire Line
-	7350 5350 7850 5350
-Wire Wire Line
-	7350 6050 7350 5950
-Wire Wire Line
-	7350 4850 7350 4650
-$Comp
-L power:+5V #PWR011
+Wire Wire Line
+	7500 5100 8000 5100
+$Comp
+L power:+5V #PWR012
 U 1 1 5FE406C7
 P 7350 4650
-F 0 "#PWR011" H 7350 4500 50  0001 C CNN
+F 0 "#PWR012" H 7350 4500 50  0001 C CNN
 F 1 "+5V" H 7365 4823 50  0000 C CNN
 F 2 "" H 7350 4650 50  0001 C CNN
@@
 $EndComp
 $Comp
-L power:GND #PWR012
+L power:GND #PWR013
 U 1 1 5FE3F7F2
-P 7350 6050
-F 0 "#PWR012" H 7350 5800 50  0001 C CNN
-F 1 "GND" H 7355 5877 50  0000 C CNN
-F 2 "" H 7350 6050 50  0001 C CNN
-F 3 "" H 7350 6050 50  0001 C CNN
-	1    7350 6050
-	1    0    0    -1
-$EndComp
-Wire Wire Line
-	7350 5650 7350 5350
-$Comp
-L Device:R R8
-U 1 1 5FE343DF
-P 7350 5800
-F 0 "R8" H 7280 5754 50  0000 R CNN
-F 1 "330" H 7280 5845 50  0000 R CNN
-F 2 "Resistor_THT:R_Axial_DIN0204_L3.6mm_D1.6mm_P7.62mm_Horizontal" V 7280 5800 50  0001 C CNN
-F 3 "~" H 7350 5800 50  0001 C CNN
-	1    7350 5800
-	-1   0    0    1
-$EndComp
-$Comp
-L Device:R R7
-U 1 1 5FE337C9
-P 7350 5000
-F 0 "R7" H 7280 4954 50  0000 R CNN
-F 1 "1k" H 7280 5045 50  0000 R CNN
-F 2 "Resistor_THT:R_Axial_DIN0204_L3.6mm_D1.6mm_P7.62mm_Horizontal" V 7280 5000 50  0001 C CNN
-F 3 "~" H 7350 5000 50  0001 C CNN
-	1    7350 5000
-	-1   0    0    1
+P 7350 5600
+F 0 "#PWR013" H 7350 5350 50  0001 C CNN
+F 1 "GND" H 7355 5427 50  0000 C CNN
+F 2 "" H 7350 5600 50  0001 C CNN
+F 3 "" H 7350 5600 50  0001 C CNN
+	1    7350 5600
+	1    0    0    -1
 $EndComp
 NoConn ~ 3100 5350
@@
 Connection ~ 2600 6300
 $Comp
-L power:GND #PWR07
+L power:GND #PWR08
 U 1 1 5FDD78C1
 P 4900 6350
-F 0 "#PWR07" H 4900 6100 50  0001 C CNN
+F 0 "#PWR08" H 4900 6100 50  0001 C CNN
 F 1 "GND" H 4905 6177 50  0000 C CNN
 F 2 "" H 4900 6350 50  0001 C CNN
@@
 Connection ~ 4900 6300
 $Comp
-L power:+5V #PWR06
+L power:+5V #PWR07
 U 1 1 5FDDA414
 P 4850 4500
-F 0 "#PWR06" H 4850 4350 50  0001 C CNN
+F 0 "#PWR07" H 4850 4350 50  0001 C CNN
 F 1 "+5V" H 4865 4673 50  0000 C CNN
 F 2 "" H 4850 4500 50  0001 C CNN
@@
 NoConn ~ 3200 5950
 $Comp
-L power:GND #PWR05
+L power:GND #PWR06
 U 1 1 5FE27632
 P 4400 5000
-F 0 "#PWR05" H 4400 4750 50  0001 C CNN
+F 0 "#PWR06" H 4400 4750 50  0001 C CNN
 F 1 "GND" H 4405 4827 50  0000 C CNN
 F 2 "" H 4400 5000 50  0001 C CNN
@@
 	6600 3200 6600 3250
 $Comp
-L power:GND #PWR09
+L power:GND #PWR010
 U 1 1 5FDC762A
 P 6600 3250
-F 0 "#PWR09" H 6600 3000 50  0001 C CNN
+F 0 "#PWR010" H 6600 3000 50  0001 C CNN
 F 1 "GND" H 6605 3077 50  0000 C CNN
 F 2 "" H 6600 3250 50  0001 C CNN
@@
 $EndComp
 $Comp
-L power:+3V3 #PWR08
+L power:+3V3 #PWR09
 U 1 1 5FDC6D0D
 P 6600 2850
-F 0 "#PWR08" H 6600 2700 50  0001 C CNN
+F 0 "#PWR09" H 6600 2700 50  0001 C CNN
 F 1 "+3V3" H 6615 3023 50  0000 C CNN
 F 2 "" H 6600 2850 50  0001 C CNN
@@
 	0    1    1    0
 $EndComp
-NoConn ~ 10550 2400
 Wire Wire Line
 	4900 5650 4900 5450
@@
 	1950 2650 1950 2550
 $Comp
-L power:GND #PWR03
+L power:GND #PWR02
 U 1 1 5FE11FE2
 P 1950 2650
-F 0 "#PWR03" H 1950 2400 50  0001 C CNN
+F 0 "#PWR02" H 1950 2400 50  0001 C CNN
 F 1 "GND" H 1955 2477 50  0000 C CNN
 F 2 "" H 1950 2650 50  0001 C CNN
@@
 $EndComp
 $Comp
-L power:GND #PWR02
+L power:GND #PWR04
 U 1 1 5FE03D4E
 P 2200 2250
-F 0 "#PWR02" H 2200 2000 50  0001 C CNN
+F 0 "#PWR04" H 2200 2000 50  0001 C CNN
 F 1 "GND" H 2205 2077 50  0000 C CNN
 F 2 "" H 2200 2250 50  0001 C CNN
@@
 $EndComp
 $Comp
-L power:+5V #PWR01
+L power:+5V #PWR03
 U 1 1 5FDFFBE4
 P 2200 1600
-F 0 "#PWR01" H 2200 1450 50  0001 C CNN
+F 0 "#PWR03" H 2200 1450 50  0001 C CNN
 F 1 "+5V" H 2215 1773 50  0000 C CNN
 F 2 "" H 2200 1600 50  0001 C CNN
@@
 $EndComp
 $Comp
-L power:+5V #PWR0101
+L power:+5V #PWR01
 U 1 1 5FE90111
 P 1950 2450
-F 0 "#PWR0101" H 1950 2300 50  0001 C CNN
+F 0 "#PWR01" H 1950 2300 50  0001 C CNN
 F 1 "+5V" H 1965 2623 50  0000 C CNN
 F 2 "" H 1950 2450 50  0001 C CNN
@@
 Wire Wire Line
 	1950 2550 2600 2550
+$Comp
+L Device:R_POT RV1
+U 1 1 5FD6B59A
+P 7350 5100
+F 0 "RV1" H 7281 5146 50  0000 R CNN
+F 1 "R_POT" H 7281 5055 50  0000 R CNN
+F 2 "Potentiometer_THT:Potentiometer_ACP_CA9-V10_Vertical" H 7350 5100 50  0001 C CNN
+F 3 "~" H 7350 5100 50  0001 C CNN
+	1    7350 5100
+	1    0    0    -1
+$EndComp
+Wire Wire Line
+	7350 4950 7350 4650
+Text Label 8000 5100 0    50   ~ 0
+D6(**)
+Wire Wire Line
+	7350 5250 7350 5600
 $EndSCHEMATC
